File: samsung_regulator/samsung_regulator.kicad_pcb (KiCad board)
At the start: 2 copper layers, 9 parts, among them K1 CONN_3

Commit message: update
Parts:
- R2: footprint 3PIN_6mm -> CVAR3X2
- moved R3 132.2 mm to (205.7, 100.3), turned to 270 degrees
- moved R1 97.3 mm to (190.5, 106.7), turned to 180 degrees
- moved COUT1 88.5 mm to (188.0, 111.8), turned to 180 degrees
- moved CIN1 84.7 mm to (182.9, 100.3)
- moved CF1 73.3 mm to (181.6, 73.7), turned to 180 degrees
- moved K1 34.1 mm to (186.7, 118.1)
- moved R2 20.9 mm to (203.2, 86.4)
- moved R4 6.48 mm to (185.4, 90.2)
Routing:
- net N-000006: track 0.00 -> 157.9 mm
- net GND: track 0.00 -> 59.6 mm
- net N-000007: track 0.00 -> 51.1 mm
- net N-000003: track 0.00 -> 22.1 mm
- net N-000005: track 0.00 -> 12.5 mm
- net N-000004: track 0.00 -> 6.35 mm
- net N-000002: track 0.00 -> 5.08 mm

Commit message: update
Parts:
- moved R3 6.48 mm to (199.4, 99.1)
- moved R2 6.48 mm to (196.8, 85.1)
Routing:
- net N-000006: track 157.9 -> 127.2 mm
- net N-000005: track 12.5 -> 0.00 mm
Changed lines of the file:
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@@
   (general
     (links 15)
-    (no_connects 2)
-    (area 0 0 0 0)
+    (no_connects 3)
+    (area 175.468845 42.98982 202.336401 124.3584)
     (thickness 1.6)
     (drawings 0)
-    (tracks 37)
+    (tracks 34)
     (zones 0)
     (modules 9)
@@
   )
   (module R3 (layer F.Cu)
-    (at 205.74 100.33 270)
+    (at 199.39 99.06 270)
     (descr "Resitance 3 pas")
     (tags R)
@@
   )
   (module CVAR3X2 (layer F.Cu)
-    (at 203.2 86.36)
+    (at 196.85 85.09)
     (descr "Condensateur ajustable")
     (tags "C DEV")
@@
   (segment (start 190.5 76.2) (end 190.5 68.58) (width 0.254) (layer B.Cu) (net 3))
   (segment (start 189.23 77.47) (end 190.5 76.2) (width 0.254) (layer B.Cu) (net 3))
-  (segment (start 205.74 96.52) (end 205.74 90.17) (width 0.254) (layer B.Cu) (net 4) (status C00000))
-  (segment (start 194.31 106.68) (end 203.2 106.68) (width 0.254) (layer B.Cu) (net 5) (status 400000))
-  (segment (start 203.2 106.68) (end 205.74 104.14) (width 0.254) (layer B.Cu) (net 5) (status 800000))
-  (segment (start 182.88 68.58) (end 182.88 73.66) (width 0.254) (layer B.Cu) (net 6) (status C00000))
-  (segment (start 203.2 82.55) (end 203.2 64.77) (width 0.254) (layer B.Cu) (net 6) (status 400000))
-  (segment (start 203.2 64.77) (end 201.93 63.5) (width 0.254) (layer B.Cu) (net 6))
-  (segment (start 201.93 63.5) (end 182.88 63.5) (width 0.254) (layer B.Cu) (net 6))
-  (segment (start 182.88 63.5) (end 182.88 68.58) (width 0.254) (layer B.Cu) (net 6) (status 800000))
+  (segment (start 199.39 95.25) (end 199.39 88.9) (width 0.254) (layer B.Cu) (net 4))
+  (segment (start 196.85 81.28) (end 196.85 68.58) (width 0.254) (layer B.Cu) (net 6))
+  (segment (start 185.42 66.04) (end 182.88 68.58) (width 0.254) (layer B.Cu) (net 6))
+  (segment (start 194.31 66.04) (end 185.42 66.04) (width 0.254) (layer B.Cu) (net 6))
+  (segment (start 196.85 68.58) (end 194.31 66.04) (width 0.254) (layer B.Cu) (net 6))
+  (segment (start 182.88 68.58) (end 182.88 73.66) (width 0.254) (layer B.Cu) (net 6))
+  (segment (start 182.88 63.5) (end 182.88 68.58) (width 0.254) (layer B.Cu) (net 6))
   (segment (start 182.88 68.58) (end 182.88 63.5) (width 0.254) (layer B.Cu) (net 6))
-  (segment (start 201.93 63.5) (end 203.2 64.77) (width 0.254) (layer B.Cu) (net 6))
-  (segment (start 182.88 63.5) (end 201.93 63.5) (width 0.254) (layer B.Cu) (net 6))
   (segment (start 189.23 111.76) (end 189.23 115.57) (width 0.254) (layer B.Cu) (net 6))
   (segment (start 189.23 115.57) (end 191.77 118.11) (width 0.254) (layer B.Cu) (net 6))

Commit message: connected all
Routing:
- net N-000007: track 51.1 -> 61.3 mm
- net N-000005: track 0.00 -> 6.66 mm
- net GND: track 59.6 -> 65.9 mm
Changed lines of the file:
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@@
   (general
     (links 15)
-    (no_connects 3)
+    (no_connects 0)
     (area 175.468845 42.98982 202.336401 124.3584)
     (thickness 1.6)
     (drawings 0)
-    (tracks 34)
+    (tracks 38)
     (zones 0)
     (modules 9)
@@
     )
   )
+  (segment (start 186.69 118.11) (end 186.69 111.76) (width 0.254) (layer B.Cu) (net 1))
   (segment (start 186.69 106.68) (end 186.69 102.87) (width 0.254) (layer B.Cu) (net 1))
   (segment (start 186.69 102.87) (end 184.15 100.33) (width 0.254) (layer B.Cu) (net 1))
@@
   (segment (start 189.23 77.47) (end 190.5 76.2) (width 0.254) (layer B.Cu) (net 3))
   (segment (start 199.39 95.25) (end 199.39 88.9) (width 0.254) (layer B.Cu) (net 4))
+  (segment (start 194.31 106.68) (end 195.58 106.68) (width 0.254) (layer B.Cu) (net 5))
+  (segment (start 195.58 106.68) (end 199.39 102.87) (width 0.254) (layer B.Cu) (net 5))
   (segment (start 196.85 81.28) (end 196.85 68.58) (width 0.254) (layer B.Cu) (net 6))
   (segment (start 185.42 66.04) (end 182.88 68.58) (width 0.254) (layer B.Cu) (net 6))
@@
   (segment (start 177.8 123.19) (end 177.8 80.01) (width 0.254) (layer B.Cu) (net 6))
   (segment (start 191.77 123.19) (end 177.8 123.19) (width 0.254) (layer B.Cu) (net 6))
+  (segment (start 181.61 100.33) (end 181.61 90.17) (width 0.254) (layer B.Cu) (net 7))
   (segment (start 181.61 118.11) (end 181.61 100.33) (width 0.254) (layer B.Cu) (net 7))
   (segment (start 181.61 100.33) (end 181.61 80.01) (width 0.254) (layer B.Cu) (net 7))

Commit message: repositioned all
Parts:
- moved R3 37.1 mm to (170.2, 76.2), turned to 90 degrees
- moved R1 33.6 mm to (184.2, 73.7), turned to 0 degrees
- moved R2 24.3 mm to (172.7, 87.6), turned to 180 degrees
- moved K1 20.4 mm to (185.4, 97.8), turned to 180 degrees
- moved CIN1 13.7 mm to (188.0, 87.6)
- moved R4 12.5 mm to (190.5, 78.7)
- moved CF1 6.35 mm to (181.6, 80.0)
- moved COUT1 2.84 mm to (186.7, 109.2), turned to 0 degrees
Connections:
- CF1 pad 2: N-000002 (its old number) -> N-000005
- K1 pad 1: N-000007 -> GND
- K1 pad 2: GND -> N-000007
- R5 pad 5: N-000002 (its old number) -> N-000005
Routing:
- net N-000006: track 127.2 -> 0.00 mm
- net GND: track 65.9 -> 0.00 mm
- net N-000007: track 61.3 -> 0.00 mm
- net N-000002: track 22.1 -> 0.00 mm
- net N-000005: track 6.66 -> 0.00 mm
- net N-000001: track 6.35 -> 0.00 mm
- net N-000002 (its old number): track 5.08 -> 0.00 mm

Commit message: linked
Parts:
- moved COUT1 46.2 mm to (174.0, 64.8), turned to 90 degrees
- moved CF1 2.54 mm to (181.6, 82.5)
- moved CIN1 1.27 mm to (186.7, 87.6)
- moved R2 1.27 mm to (172.7, 88.9)
- moved R4 1.27 mm to (189.2, 78.7)
- moved R3 1.27 mm to (170.2, 77.5)
Routing:
- net N-000006: track 0.00 -> 52.9 mm
- net GND: track 0.00 -> 46.3 mm
- net N-000007: track 0.00 -> 29.2 mm
- net N-000005: track 0.00 -> 24.1 mm
- net N-000002: track 0.00 -> 11.2 mm
- net N-000001: track 0.00 -> 3.81 mm
Changed lines of the file:
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@@
   (general
     (links 16)
-    (no_connects 16)
+    (no_connects 1)
     (area 131.673599 42.98982 230.276401 127.406401)
     (thickness 1.6)
     (drawings 0)
-    (tracks 0)
+    (tracks 21)
     (zones 0)
     (modules 9)
@@
   )
   (module R3 (layer F.Cu)
-    (at 170.18 76.2 90)
+    (at 170.18 77.47 90)
     (descr "Resitance 3 pas")
     (tags R)
@@
   )
   (module R3 (layer F.Cu)
-    (at 190.5 78.74)
+    (at 189.23 78.74)
     (descr "Resitance 3 pas")
     (tags R)
@@
   )
   (module C1 (layer F.Cu)
-    (at 187.96 87.63)
+    (at 186.69 87.63)
     (descr "Condensateur e = 1 pas")
     (tags C)
@@
   )
   (module C1 (layer F.Cu)
-    (at 181.61 80.01 180)
+    (at 181.61 82.55 180)
     (descr "Condensateur e = 1 pas")
     (tags C)
@@
   )
   (module C1 (layer F.Cu)
-    (at 186.69 109.22)
+    (at 173.99 64.77 90)
     (descr "Condensateur e = 1 pas")
     (tags C)
-    (fp_text reference COUT1 (at 0.254 -2.286) (layer F.SilkS)
-      (effects (font (size 1.016 1.016) (thickness 0.2032)))
-    )
-    (fp_text value C (at 0 -2.286) (layer F.SilkS) hide
+    (fp_text reference COUT1 (at 0.254 -2.286 90) (layer F.SilkS)
+      (effects (font (size 1.016 1.016) (thickness 0.2032)))
+    )
+    (fp_text value C (at 0 -2.286 90) (layer F.SilkS) hide
       (effects (font (size 1.016 1.016) (thickness 0.2032)))
     )
@@
     (fp_line (start -2.54 1.27) (end -2.54 -1.27) (layer F.SilkS) (width 0.3048))
     (fp_line (start -2.54 -0.635) (end -1.905 -1.27) (layer F.SilkS) (width 0.3048))
-    (pad 1 thru_hole circle (at -1.27 0) (size 1.397 1.397) (drill 0.8128)
+    (pad 1 thru_hole circle (at -1.27 0 90) (size 1.397 1.397) (drill 0.8128)
       (layers *.Cu *.Mask F.SilkS)
       (net 5 N-000006)
     )
-    (pad 2 thru_hole circle (at 1.27 0) (size 1.397 1.397) (drill 0.8128)
+    (pad 2 thru_hole circle (at 1.27 0 90) (size 1.397 1.397) (drill 0.8128)
       (layers *.Cu *.Mask F.SilkS)
       (net 1 GND)
@@
   )
   (module CVAR3X2 (layer F.Cu)
-    (at 172.72 87.63 180)
+    (at 172.72 88.9 180)
     (descr "Condensateur ajustable")
     (tags "C DEV")
@@
     )
   )
+  (segment (start 190.5 97.79) (end 190.5 90.17) (width 0.254) (layer B.Cu) (net 1))
+  (segment (start 190.5 90.17) (end 187.96 87.63) (width 0.254) (layer B.Cu) (net 1))
+  (segment (start 187.96 87.63) (end 187.96 68.58) (width 0.254) (layer B.Cu) (net 1))
+  (segment (start 173.99 63.5) (end 182.88 63.5) (width 0.254) (layer B.Cu) (net 1))
+  (segment (start 182.88 63.5) (end 187.96 68.58) (width 0.254) (layer B.Cu) (net 1))
+  (segment (start 170.18 81.28) (end 170.18 85.09) (width 0.254) (layer B.Cu) (net 2))
+  (segment (start 193.04 78.74) (end 193.04 71.12) (width 0.254) (layer B.Cu) (net 3))
+  (segment (start 193.04 71.12) (end 190.5 68.58) (width 0.254) (layer B.Cu) (net 3))
+  (segment (start 180.34 73.66) (end 180.34 82.55) (width 0.254) (layer B.Cu) (net 4) (status 20))
+  (segment (start 180.34 73.66) (end 180.34 68.58) (width 0.254) (layer B.Cu) (net 4))
+  (segment (start 170.18 73.66) (end 180.34 73.66) (width 0.254) (layer B.Cu) (net 4))
+  (segment (start 182.88 82.55) (end 182.88 68.58) (width 0.254) (layer B.Cu) (net 5) (status C00000))
+  (segment (start 182.88 82.55) (end 182.88 95.25) (width 0.254) (layer B.Cu) (net 5) (status 10))
+  (segment (start 182.88 95.25) (end 180.34 97.79) (width 0.254) (layer B.Cu) (net 5))
+  (segment (start 172.72 92.71) (end 172.72 97.79) (width 0.254) (layer B.Cu) (net 5))
+  (segment (start 172.72 97.79) (end 180.34 97.79) (width 0.254) (layer B.Cu) (net 5))
+  (segment (start 173.99 66.04) (end 180.34 66.04) (width 0.254) (layer B.Cu) (net 5))
+  (segment (start 180.34 66.04) (end 182.88 68.58) (width 0.254) (layer B.Cu) (net 5))
+  (segment (start 185.42 97.79) (end 185.42 87.63) (width 0.254) (layer B.Cu) (net 6))
+  (segment (start 185.42 87.63) (end 185.42 78.74) (width 0.254) (layer B.Cu) (net 6))
+  (segment (start 185.42 78.74) (end 185.42 68.58) (width 0.254) (layer B.Cu) (net 6))
 )

Commit message: up
Parts:
- COUT1: footprint C1 -> C2
- R2: footprint CVAR3X2 -> RVAR
- moved COUT1 12.0 mm to (185.4, 68.6), turned to 0 degrees
- moved R5 5.08 mm to (185.4, 61.0)
- moved R3 3.81 mm to (174.0, 77.5)
- moved R2 1.80 mm to (171.4, 90.2)
Routing:
- net GND: track 46.3 -> 35.3 mm
- net N-000006: track 29.2 -> 34.3 mm
- net N-000003: track 11.2 -> 16.3 mm
- net N-000004: track 52.9 -> 48.0 mm
- net N-000005: track 24.1 -> 25.4 mm
- net N-000002: track 3.81 -> 5.08 mm

Commit message: up
Parts:
- moved CF1 7.62 mm to (181.6, 90.2)
- moved R5 7.62 mm to (185.4, 68.6)
- moved COUT1 6.35 mm to (185.4, 74.9)
- moved R1 5.08 mm to (184.2, 78.7)
- moved R4 3.81 mm to (189.2, 82.5)
- moved R2 2.84 mm to (172.7, 87.6)
- moved R3 2.84 mm to (175.3, 74.9)
- moved CIN1 1.27 mm to (186.7, 86.4)
Routing:
- net GND: track 35.3 -> 27.4 mm
- net N-000004: track 48.0 -> 40.2 mm
- net N-000006: track 34.3 -> 26.7 mm
- net N-000005: track 25.4 -> 19.0 mm
- net N-000003: track 16.3 -> 12.5 mm
Changed lines of the file:
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@@
   (general
     (links 16)
-    (no_connects 0)
-    (area 162.153599 37.90982 195.371155 104.0384)
+    (no_connects 1)
+    (area 167.233599 45.52982 195.371155 104.0384)
     (thickness 1.6)
     (drawings 0)
-    (tracks 20)
+    (tracks 22)
     (zones 0)
     (modules 9)
@@
   )
   (module TO220-5 (layer F.Cu)
-    (at 185.42 60.96 90)
+    (at 185.42 68.58 90)
     (descr "Transistor TO 220-5")
     (tags "TR TO220 DEV")
@@
   )
   (module R3 (layer F.Cu)
-    (at 184.15 73.66)
+    (at 184.15 78.74)
     (descr "Resitance 3 pas")
     (tags R)
@@
   )
   (module R3 (layer F.Cu)
-    (at 173.99 77.47 90)
+    (at 175.26 74.93 90)
     (descr "Resitance 3 pas")
     (tags R)
@@
   )
   (module R3 (layer F.Cu)
-    (at 189.23 78.74)
+    (at 189.23 82.55)
     (descr "Resitance 3 pas")
     (tags R)
@@
   )
   (module C1 (layer F.Cu)
-    (at 186.69 87.63)
+    (at 186.69 86.36)
     (descr "Condensateur e = 1 pas")
     (tags C)
@@
   )
   (module C1 (layer F.Cu)
-    (at 181.61 82.55 180)
+    (at 181.61 90.17 180)
     (descr "Condensateur e = 1 pas")
     (tags C)
@@
   )
   (module C2 (layer F.Cu)
-    (at 185.42 68.58)
+    (at 185.42 74.93)
     (descr "Condensateur = 2 pas")
     (tags C)
@@
   )
   (module RVAR (layer F.Cu)
-    (at 171.45 90.17 180)
+    (at 172.72 87.63 180)
     (descr "Resistance variable")
     (tags RV)
@@
     )
   )
-  (segment (start 187.96 63.5) (end 187.96 68.58) (width 0.254) (layer B.Cu) (net 1))
-  (segment (start 187.96 68.58) (end 187.96 73.66) (width 0.254) (layer B.Cu) (net 1))
-  (segment (start 187.96 73.66) (end 187.96 87.63) (width 0.254) (layer B.Cu) (net 1))
+  (segment (start 187.96 71.12) (end 187.96 74.93) (width 0.254) (layer B.Cu) (net 1))
+  (segment (start 187.96 74.93) (end 187.96 78.74) (width 0.254) (layer B.Cu) (net 1) (status 10))
+  (segment (start 187.96 78.74) (end 187.96 86.36) (width 0.254) (layer B.Cu) (net 1) (status 10))
   (segment (start 190.5 97.79) (end 190.5 90.17) (width 0.254) (layer B.Cu) (net 1))
-  (segment (start 190.5 90.17) (end 187.96 87.63) (width 0.254) (layer B.Cu) (net 1))
-  (segment (start 173.99 86.36) (end 173.99 81.28) (width 0.254) (layer B.Cu) (net 2) (status 20))
-  (segment (start 193.04 78.74) (end 193.04 66.04) (width 0.254) (layer B.Cu) (net 3))
-  (segment (start 193.04 66.04) (end 190.5 63.5) (width 0.254) (layer B.Cu) (net 3))
-  (segment (start 180.34 97.79) (end 171.45 97.79) (width 0.254) (layer B.Cu) (net 4))
-  (segment (start 171.45 97.79) (end 171.45 93.98) (width 0.254) (layer B.Cu) (net 4) (status 20))
-  (segment (start 182.88 63.5) (end 182.88 68.58) (width 0.254) (layer B.Cu) (net 4))
-  (segment (start 182.88 68.58) (end 182.88 82.55) (width 0.254) (layer B.Cu) (net 4) (status 20))
-  (segment (start 182.88 82.55) (end 182.88 95.25) (width 0.254) (layer B.Cu) (net 4) (status 10))
+  (segment (start 190.5 90.17) (end 187.96 86.36) (width 0.254) (layer B.Cu) (net 1) (status 20))
+  (segment (start 175.26 83.82) (end 175.26 80.01) (width 0.254) (layer B.Cu) (net 2))
+  (segment (start 175.26 80.01) (end 175.26 78.74) (width 0.254) (layer B.Cu) (net 2) (status 20))
+  (segment (start 190.5 71.12) (end 193.04 73.66) (width 0.254) (layer B.Cu) (net 3))
+  (segment (start 193.04 73.66) (end 193.04 82.55) (width 0.254) (layer B.Cu) (net 3))
+  (segment (start 172.72 91.44) (end 172.72 95.25) (width 0.254) (layer B.Cu) (net 4))
+  (segment (start 175.26 97.79) (end 180.34 97.79) (width 0.254) (layer B.Cu) (net 4))
+  (segment (start 172.72 95.25) (end 175.26 97.79) (width 0.254) (layer B.Cu) (net 4))
+  (segment (start 182.88 74.93) (end 182.88 71.12) (width 0.254) (layer B.Cu) (net 4))
+  (segment (start 182.88 74.93) (end 182.88 90.17) (width 0.254) (layer B.Cu) (net 4) (status 10))
+  (segment (start 182.88 90.17) (end 182.88 95.25) (width 0.254) (layer B.Cu) (net 4) (status 10))
   (segment (start 182.88 95.25) (end 180.34 97.79) (width 0.254) (layer B.Cu) (net 4))
-  (segment (start 173.99 73.66) (end 180.34 73.66) (width 0.254) (layer B.Cu) (net 5) (status 10))
-  (segment (start 180.34 73.66) (end 180.34 63.5) (width 0.254) (layer B.Cu) (net 5))
-  (segment (start 180.34 73.66) (end 180.34 82.55) (width 0.254) (layer B.Cu) (net 5) (status 20))
-  (segment (start 185.42 63.5) (end 185.42 78.74) (width 0.254) (layer B.Cu) (net 6))
-  (segment (start 185.42 97.79) (end 185.42 87.63) (width 0.254) (layer B.Cu) (net 6))
-  (segment (start 185.42 87.63) (end 185.42 78.74) (width 0.254) (layer B.Cu) (net 6))
+  (segment (start 180.34 78.74) (end 180.34 71.12) (width 0.254) (layer B.Cu) (net 5))
+  (segment (start 180.34 90.17) (end 180.34 82.55) (width 0.254) (layer B.Cu) (net 5) (status 20))
+  (segment (start 180.34 82.55) (end 180.34 78.74) (width 0.254) (layer B.Cu) (net 5) (status 10))
+  (segment (start 185.42 82.55) (end 185.42 71.12) (width 0.254) (layer B.Cu) (net 6))
+  (segment (start 185.42 97.79) (end 185.42 86.36) (width 0.254) (layer B.Cu) (net 6) (status 20))
+  (segment (start 185.42 86.36) (end 185.42 82.55) (width 0.254) (layer B.Cu) (net 6) (status 10))
 )

Commit message: thinker tracks
Routing:
- net N-000005: track 19.0 -> 24.1 mm
Other:
- board outline added: 27.9 x 33 mm
- net class Default: clearance 0.254 -> 0.8; trace_width 0.254 -> 0.8
- rule trace_clearance: 0.254 -> 0.8
- rule trace_min: 0.254 -> 0.8
Changed lines of the file:
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@@
   (general
     (links 16)
-    (no_connects 1)
+    (no_connects 0)
     (area 167.233599 45.52982 195.371155 104.0384)
     (thickness 1.6)
-    (drawings 0)
-    (tracks 22)
+    (drawings 4)
+    (tracks 23)
     (zones 0)
     (modules 9)
@@
   )
   (setup
-    (last_trace_width 0.254)
-    (trace_clearance 0.254)
+    (last_trace_width 0.8)
+    (trace_clearance 0.8)
     (zone_clearance 0.508)
     (zone_45_only no)
-    (trace_min 0.254)
+    (trace_min 0.8)
     (segment_width 0.2)
     (edge_width 0.15)
@@
   (net 6 N-000006)
   (net_class Default "This is the default net class."
-    (clearance 0.254)
-    (trace_width 0.254)
+    (clearance 0.8)
+    (trace_width 0.8)
     (via_dia 0.889)
     (via_drill 0.635)
@@
     )
   )
-  (segment (start 187.96 71.12) (end 187.96 74.93) (width 0.254) (layer B.Cu) (net 1))
-  (segment (start 187.96 74.93) (end 187.96 78.74) (width 0.254) (layer B.Cu) (net 1) (status 10))
-  (segment (start 187.96 78.74) (end 187.96 86.36) (width 0.254) (layer B.Cu) (net 1) (status 10))
-  (segment (start 190.5 97.79) (end 190.5 90.17) (width 0.254) (layer B.Cu) (net 1))
-  (segment (start 190.5 90.17) (end 187.96 86.36) (width 0.254) (layer B.Cu) (net 1) (status 20))
-  (segment (start 175.26 83.82) (end 175.26 80.01) (width 0.254) (layer B.Cu) (net 2))
-  (segment (start 175.26 80.01) (end 175.26 78.74) (width 0.254) (layer B.Cu) (net 2) (status 20))
-  (segment (start 190.5 71.12) (end 193.04 73.66) (width 0.254) (layer B.Cu) (net 3))
-  (segment (start 193.04 73.66) (end 193.04 82.55) (width 0.254) (layer B.Cu) (net 3))
-  (segment (start 172.72 91.44) (end 172.72 95.25) (width 0.254) (layer B.Cu) (net 4))
-  (segment (start 175.26 97.79) (end 180.34 97.79) (width 0.254) (layer B.Cu) (net 4))
-  (segment (start 172.72 95.25) (end 175.26 97.79) (width 0.254) (layer B.Cu) (net 4))
-  (segment (start 182.88 74.93) (end 182.88 71.12) (width 0.254) (layer B.Cu) (net 4))
-  (segment (start 182.88 74.93) (end 182.88 90.17) (width 0.254) (layer B.Cu) (net 4) (status 10))
-  (segment (start 182.88 90.17) (end 182.88 95.25) (width 0.254) (layer B.Cu) (net 4) (status 10))
-  (segment (start 182.88 95.25) (end 180.34 97.79) (width 0.254) (layer B.Cu) (net 4))
-  (segment (start 180.34 78.74) (end 180.34 71.12) (width 0.254) (layer B.Cu) (net 5))
-  (segment (start 180.34 90.17) (end 180.34 82.55) (width 0.254) (layer B.Cu) (net 5) (status 20))
-  (segment (start 180.34 82.55) (end 180.34 78.74) (width 0.254) (layer B.Cu) (net 5) (status 10))
-  (segment (start 185.42 82.55) (end 185.42 71.12) (width 0.254) (layer B.Cu) (net 6))
-  (segment (start 185.42 97.79) (end 185.42 86.36) (width 0.254) (layer B.Cu) (net 6) (status 20))
-  (segment (start 185.42 86.36) (end 185.42 82.55) (width 0.254) (layer B.Cu) (net 6) (status 10))
+  (gr_line (start 195.58 68.58) (end 195.58 101.6) (angle 90) (layer Edge.Cuts) (width 0.15))
+  (gr_line (start 167.64 68.58) (end 195.58 68.58) (angle 90) (layer Edge.Cuts) (width 0.15))
+  (gr_line (start 167.64 101.6) (end 167.64 68.58) (angle 90) (layer Edge.Cuts) (width 0.15))
+  (gr_line (start 195.58 101.6) (end 167.64 101.6) (angle 90) (layer Edge.Cuts) (width 0.15))
+  (segment (start 187.96 71.12) (end 187.96 74.93) (width 0.8) (layer B.Cu) (net 1))
+  (segment (start 187.96 74.93) (end 187.96 78.74) (width 0.8) (layer B.Cu) (net 1) (status 10))
+  (segment (start 187.96 78.74) (end 187.96 86.36) (width 0.8) (layer B.Cu) (net 1) (status 10))
+  (segment (start 190.5 97.79) (end 190.5 90.17) (width 0.8) (layer B.Cu) (net 1))
+  (segment (start 190.5 90.17) (end 187.96 86.36) (width 0.8) (layer B.Cu) (net 1) (status 20))
+  (segment (start 175.26 83.82) (end 175.26 80.01) (width 0.8) (layer B.Cu) (net 2))
+  (segment (start 175.26 80.01) (end 175.26 78.74) (width 0.8) (layer B.Cu) (net 2) (status 20))
+  (segment (start 190.5 71.12) (end 193.04 73.66) (width 0.8) (layer B.Cu) (net 3))
+  (segment (start 193.04 73.66) (end 193.04 82.55) (width 0.8) (layer B.Cu) (net 3))
+  (segment (start 172.72 91.44) (end 172.72 95.25) (width 0.8) (layer B.Cu) (net 4))
+  (segment (start 175.26 97.79) (end 180.34 97.79) (width 0.8) (layer B.Cu) (net 4))
+  (segment (start 172.72 95.25) (end 175.26 97.79) (width 0.8) (layer B.Cu) (net 4))
+  (segment (start 182.88 74.93) (end 182.88 71.12) (width 0.8) (layer B.Cu) (net 4))
+  (segment (start 182.88 74.93) (end 182.88 90.17) (width 0.8) (layer B.Cu) (net 4) (status 10))
+  (segment (start 182.88 90.17) (end 182.88 95.25) (width 0.8) (layer B.Cu) (net 4) (status 10))
+  (segment (start 182.88 95.25) (end 180.34 97.79) (width 0.8) (layer B.Cu) (net 4))
+  (segment (start 175.26 71.12) (end 180.34 71.12) (width 0.8) (layer B.Cu) (net 5) (status C00000))
+  (segment (start 180.34 78.74) (end 180.34 71.12) (width 0.8) (layer B.Cu) (net 5))
+  (segment (start 180.34 90.17) (end 180.34 82.55) (width 0.8) (layer B.Cu) (net 5) (status 20))
+  (segment (start 180.34 82.55) (end 180.34 78.74) (width 0.8) (layer B.Cu) (net 5) (status 10))
+  (segment (start 185.42 82.55) (end 185.42 71.12) (width 0.8) (layer B.Cu) (net 6))
+  (segment (start 185.42 97.79) (end 185.42 86.36) (width 0.8) (layer B.Cu) (net 6) (status 20))
+  (segment (start 185.42 86.36) (end 185.42 82.55) (width 0.8) (layer B.Cu) (net 6) (status 10))
 )
