File: samsung_regulator/samsung_regulator.sch (KiCad schematic (older format))
At the start: 9 parts, among them K1 CONN_3

Commit message: repositioned all
Connections:
- net GND: now also K1.1 (P1); no longer K1.2 (PM)
- net at CIN1.1, R4.1, R5.2 (VIN): now also K1.2 (PM); no longer K1.1 (P1)
Changed lines of the file:
@@
 Sheet 1 1
 Title ""
-Date "15 sep 2014"
+Date "3 nov 2014"
 Rev ""
 Comp ""
@@
 Wire Wire Line
 	5850 3950 5850 4100
-Wire Wire Line
-	4650 1700 3300 1700
-Wire Wire Line
-	3300 1700 3300 2650
 Connection ~ 3300 2650
 Wire Wire Line
@@
 L GND #PWR05
 U 1 1 5404D9FD
-P 4750 1900
-F 0 "#PWR05" H 4750 1900 30  0001 C CNN
-F 1 "GND" H 4750 1830 30  0001 C CNN
-F 2 "" H 4750 1900 60  0000 C CNN
-F 3 "" H 4750 1900 60  0000 C CNN
-	1    4750 1900
-	1    0    0    -1
-$EndComp
-Wire Wire Line
-	4750 1700 4750 1900
+P 4650 1900
+F 0 "#PWR05" H 4650 1900 30  0001 C CNN
+F 1 "GND" H 4650 1830 30  0001 C CNN
+F 2 "" H 4650 1900 60  0000 C CNN
+F 3 "" H 4650 1900 60  0000 C CNN
+	1    4650 1900
+	1    0    0    -1
+$EndComp
+Wire Wire Line
+	4650 1700 4650 1900
 $Comp
 L PWR_FLAG #FLG06
@@
 Connection ~ 5850 3450
 Connection ~ 5350 2100
+Wire Wire Line
+	3300 2650 3300 2100
+Wire Wire Line
+	3300 2100 4750 2100
+Wire Wire Line
+	4750 2100 4750 1700
 $EndSCHEMATC

Commit message: up
Changed lines of the file:
@@
 Sheet 1 1
 Title ""
-Date "3 nov 2014"
+Date "10 nov 2014"
 Rev ""
 Comp ""
@@
 Wire Wire Line
 	5350 2350 6850 2350
-Wire Wire Line
-	5350 2900 5350 3450
-Wire Wire Line
-	5350 3450 6400 3450
 Connection ~ 6400 2350
 Wire Wire Line
@@
 Wire Wire Line
 	6850 1700 4850 1700
-Wire Wire Line
-	6400 3450 6400 2750
 Wire Wire Line
 	4700 3400 4700 3650
@@
 Connection ~ 3700 2650
 Connection ~ 5850 3450
-Connection ~ 5350 2100
 Wire Wire Line
 	3300 2650 3300 2100
@@
 Wire Wire Line
 	4750 2100 4750 1700
+Connection ~ 6400 2750
+Connection ~ 4650 1700
+Connection ~ 4750 1700
+Connection ~ 4850 1700
+Connection ~ 3300 3050
+Connection ~ 3700 3150
+Connection ~ 4050 2900
+Connection ~ 4050 2650
+Connection ~ 5350 2650
+Connection ~ 5350 2900
+Connection ~ 4700 3400
+Connection ~ 5850 2850
+Connection ~ 5850 2950
+Connection ~ 5850 3950
+Connection ~ 6850 2350
+Connection ~ 6850 2750
+Connection ~ 6850 3550
+Wire Wire Line
+	5350 2900 5350 3450
+Wire Wire Line
+	5350 3450 6400 3450
+Wire Wire Line
+	6400 3450 6400 2750
 $EndSCHEMATC

Commit message: named nets
Connections:
- net SD: now reaches R4.2, R5.1 (SD)
- net VIN: now reaches CIN1.1, K1.2 (PM), R4.1, R5.2 (VIN)
- net VOUT: now reaches CF1.1, COUT1.1, K1.3 (P3), R2.1, R5.4 (VOUT)
- net ADJ: now reaches CF1.2, R1.1, R3.2, R5.5 (ADJ)
Changed lines of the file:
@@
 Sheet 1 1
 Title ""
-Date "10 nov 2014"
+Date "16 nov 2014"
 Rev ""
 Comp ""
@@
 Wire Wire Line
 	6400 3450 6400 2750
+Text Label 4950 1700 0    60   ~ 0
+VOUT
+Text Label 4350 2100 0    60   ~ 0
+VIN
+Text Label 3900 3150 0    60   ~ 0
+SD
+Text Label 5600 3450 0    60   ~ 0
+ADJ
 $EndSCHEMATC
