File: samsung_regulator/.kicad_pcb.kicad_pcb (KiCad board)
At the start: 2 copper layers, 27.9 x 27.9 mm, 9 parts, among them K1 CONN_3

Commit message: added logos
Parts:
- added VAL: REF, sigmike, F.Cu at (170.8, 74.9)
- added VAL: REF, acolab, F.Cu at (172.7, 93.3)
Changed lines of the file:
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@@
     (links 16)
     (no_connects 0)
-    (area 166.687599 44.98382 195.917155 99.5044)
+    (area 166.687599 67.1704 195.917155 99.5044)
     (thickness 1.6)
     (drawings 4)
     (tracks 22)
     (zones 0)
-    (modules 9)
+    (modules 11)
     (nets 7)
   )
@@
     )
   )
+  (module sigmike (layer F.Cu)
+    (at 170.815 74.93)
+    (fp_text reference VAL (at 0 0) (layer F.SilkS) hide
+      (effects (font (size 0.381 0.381) (thickness 0.127)))
+    )
+    (fp_text value REF (at 0 0) (layer F.SilkS) hide
+      (effects (font (size 0.381 0.381) (thickness 0.127)))
+    )
+    (fp_poly (pts (xy 2.35458 2.86258) (xy -0.0127 2.86258) (xy -2.37744 2.86258) (xy -2.37744 2.21742)
+      (xy -2.37744 1.57226) (xy -2.13614 1.57226) (xy -1.89484 1.57226) (xy -1.89484 1.97612)
+      (xy -1.89484 2.37998) (xy -0.58166 2.37998) (xy -0.22352 2.37998) (xy 0.0635 2.37744)
+      (xy 0.28448 2.3749) (xy 0.44958 2.37236) (xy 0.56388 2.36728) (xy 0.63754 2.35966)
+      (xy 0.67818 2.3495) (xy 0.69088 2.33426) (xy 0.6858 2.31648) (xy 0.67818 2.30378)
+      (xy 0.64008 2.25552) (xy 0.55626 2.15392) (xy 0.43434 2.0066) (xy 0.2794 1.82372)
+      (xy 0.1016 1.61036) (xy -0.09652 1.37668) (xy -0.18034 1.27254) (xy -0.381 1.03632)
+      (xy -0.56388 0.81534) (xy -0.72136 0.6223) (xy -0.8509 0.46482) (xy -0.94234 0.34798)
+      (xy -0.99314 0.2794) (xy -0.99822 0.26924) (xy -0.97536 0.2286) (xy -0.90424 0.13716)
+      (xy -0.78994 -0.00254) (xy -0.63754 -0.18288) (xy -0.4572 -0.3937) (xy -0.25146 -0.63246)
+      (xy -0.0254 -0.889) (xy 0.02032 -0.94234) (xy 0.24892 -1.20142) (xy 0.45974 -1.44018)
+      (xy 0.6477 -1.65608) (xy 0.80518 -1.83642) (xy 0.92964 -1.97866) (xy 1.01092 -2.07518)
+      (xy 1.04648 -2.11836) (xy 1.04902 -2.1209) (xy 1.01092 -2.12598) (xy 0.89916 -2.12852)
+      (xy 0.72644 -2.13106) (xy 0.49784 -2.1336) (xy 0.22606 -2.13614) (xy -0.08128 -2.13614)
+      (xy -0.41656 -2.13614) (xy -0.42164 -2.13868) (xy -1.88976 -2.13868) (xy -1.90246 -1.86436)
+      (xy -1.91516 -1.59258) (xy -2.13614 -1.59258) (xy -2.35966 -1.59258) (xy -2.36982 -2.2479)
+      (xy -2.37998 -2.90322) (xy -0.01778 -2.90322) (xy 0.47244 -2.90322) (xy 0.91694 -2.90068)
+      (xy 1.3081 -2.89814) (xy 1.64338 -2.89306) (xy 1.91516 -2.88798) (xy 2.12598 -2.8829)
+      (xy 2.26314 -2.87782) (xy 2.32918 -2.86766) (xy 2.33172 -2.86512) (xy 2.30378 -2.82956)
+      (xy 2.22504 -2.73812) (xy 2.10566 -2.59842) (xy 1.94818 -2.42062) (xy 1.75768 -2.20218)
+      (xy 1.54178 -1.95834) (xy 1.30302 -1.68656) (xy 1.0795 -1.4351) (xy 0.8255 -1.15062)
+      (xy 0.59182 -0.88392) (xy 0.37846 -0.64008) (xy 0.19304 -0.42672) (xy 0.04318 -0.25146)
+      (xy -0.07112 -0.1143) (xy -0.1397 -0.02794) (xy -0.16002 0) (xy -0.13462 0.0381)
+      (xy -0.06096 0.127) (xy 0.0508 0.26162) (xy 0.2032 0.43434) (xy 0.381 0.64008)
+      (xy 0.57912 0.87122) (xy 0.79502 1.1176) (xy 1.02108 1.37414) (xy 1.25222 1.63576)
+      (xy 1.48082 1.8923) (xy 1.69926 2.13868) (xy 1.90246 2.36728) (xy 2.08534 2.56794)
+      (xy 2.23774 2.73812) (xy 2.25298 2.75082) (xy 2.35458 2.86258) (xy 2.35458 2.86258)) (layer Dwgs.User) (width 0.00254))
+  )
+  (module acolab (layer F.Cu)
+    (at 172.72 93.345)
+    (fp_text reference VAL (at 0 0) (layer F.SilkS) hide
+      (effects (font (size 0.381 0.381) (thickness 0.127)))
+    )
+    (fp_text value REF (at 0 0) (layer F.SilkS) hide
+      (effects (font (size 0.381 0.381) (thickness 0.127)))
+    )
+    (fp_poly (pts (xy 3.92684 -1.57988) (xy 3.90398 -1.33604) (xy 3.79222 -1.09474) (xy 3.7846 -1.0795)
+      (xy 3.62458 -0.90424) (xy 3.42138 -0.79502) (xy 3.3782 -0.78994) (xy 3.3782 -1.56972)
+      (xy 3.3147 -1.67894) (xy 3.2004 -1.7526) (xy 3.07594 -1.7399) (xy 2.97942 -1.66878)
+      (xy 2.91592 -1.55194) (xy 2.9337 -1.42494) (xy 3.01752 -1.3208) (xy 3.11404 -1.27)
+      (xy 3.21056 -1.28778) (xy 3.2893 -1.33604) (xy 3.37312 -1.44018) (xy 3.3782 -1.56972)
+      (xy 3.3782 -0.78994) (xy 3.16484 -0.7493) (xy 3.07594 -0.74676) (xy 2.78384 -0.74676)
+      (xy 2.11582 0.0508) (xy 1.4478 0.84582) (xy 1.6129 1.1684) (xy 1.69672 1.34366)
+      (xy 1.75006 1.48844) (xy 1.78054 1.64084) (xy 1.79578 1.83642) (xy 1.79832 1.89992)
+      (xy 1.81864 2.30632) (xy 1.45796 2.30632) (xy 1.09728 2.30632) (xy 1.0668 1.99898)
+      (xy 0.99822 1.65862) (xy 0.87122 1.3843) (xy 0.68834 1.17094) (xy 0.41656 0.98806)
+      (xy 0.17272 0.89916) (xy 0.17272 -1.16078) (xy 0.11938 -1.2827) (xy 0.0381 -1.35128)
+      (xy -0.05588 -1.39192) (xy -0.13208 -1.37922) (xy -0.19812 -1.34112) (xy -0.2921 -1.23444)
+      (xy -0.3175 -1.1049) (xy -0.27178 -0.98044) (xy -0.2159 -0.92964) (xy -0.10668 -0.86868)
+      (xy -0.01524 -0.87376) (xy 0.08382 -0.92964) (xy 0.16256 -1.03378) (xy 0.17272 -1.16078)
+      (xy 0.17272 0.89916) (xy 0.127 0.88646) (xy -0.16764 0.8636) (xy -0.45466 0.91948)
+      (xy -0.7239 1.05156) (xy -0.95504 1.25984) (xy -1.07188 1.41478) (xy -1.14046 1.54686)
+      (xy -1.18364 1.6891) (xy -1.2065 1.87452) (xy -1.21158 1.9558) (xy -1.2319 2.30632)
+      (xy -1.61036 2.30632) (xy -1.98882 2.30632) (xy -1.98882 1.99898) (xy -1.94818 1.62814)
+      (xy -1.88214 1.38938) (xy -1.778 1.0795) (xy -2.25044 0.73914) (xy -2.43078 0.6096)
+      (xy -2.5908 0.50038) (xy -2.71018 0.4191) (xy -2.77368 0.381) (xy -2.77622 0.37846)
+      (xy -2.84988 0.38354) (xy -2.96418 0.41656) (xy -2.99466 0.42926) (xy -3.06324 0.44704)
+      (xy -3.06324 -0.18796) (xy -3.1242 -0.28194) (xy -3.2512 -0.31496) (xy -3.25628 -0.31496)
+      (xy -3.36042 -0.29718) (xy -3.41122 -0.22606) (xy -3.4163 -0.2032) (xy -3.41376 -0.07112)
+      (xy -3.33756 0.01778) (xy -3.22326 0.04572) (xy -3.11912 0.00762) (xy -3.07848 -0.05588)
+      (xy -3.06324 -0.18796) (xy -3.06324 0.44704) (xy -3.21818 0.49022) (xy -3.4163 0.47244)
+      (xy -3.55854 0.4064) (xy -3.73634 0.25654) (xy -3.84048 0.07112) (xy -3.87858 -0.127)
+      (xy -3.85318 -0.32512) (xy -3.76428 -0.50292) (xy -3.62204 -0.64516) (xy -3.42392 -0.7366)
+      (xy -3.31724 -0.75692) (xy -3.08356 -0.74422) (xy -2.8829 -0.65532) (xy -2.7305 -0.50546)
+      (xy -2.63906 -0.30226) (xy -2.62128 -0.14224) (xy -2.61874 -0.07366) (xy -2.61112 -0.01524)
+      (xy -2.58064 0.0381) (xy -2.52222 0.10414) (xy -2.42824 0.18542) (xy -2.28854 0.28956)
+      (xy -2.09042 0.4318) (xy -1.8669 0.58674) (xy -1.5875 0.78232) (xy -1.36652 0.5969)
+      (xy -1.11506 0.41148) (xy -0.84836 0.2667) (xy -0.59944 0.17272) (xy -0.53086 0.15748)
+      (xy -0.42926 0.13462) (xy -0.37846 0.09652) (xy -0.36322 0.01524) (xy -0.36322 -0.09398)
+      (xy -0.3683 -0.23114) (xy -0.39878 -0.31496) (xy -0.47498 -0.38608) (xy -0.54102 -0.42926)
+      (xy -0.7239 -0.59436) (xy -0.84582 -0.81026) (xy -0.90424 -1.0541) (xy -0.89154 -1.31064)
+      (xy -0.80518 -1.55194) (xy -0.8001 -1.55956) (xy -0.65278 -1.7399) (xy -0.44704 -1.87706)
+      (xy -0.21082 -1.95834) (xy 0.01778 -1.97104) (xy 0.28702 -1.89992) (xy 0.50546 -1.75768)
+      (xy 0.66294 -1.55702) (xy 0.75184 -1.3081) (xy 0.76962 -1.12776) (xy 0.75692 -0.97282)
+      (xy 0.73406 -0.84328) (xy 0.71628 -0.79756) (xy 0.6096 -0.64262) (xy 0.45974 -0.49022)
+      (xy 0.30734 -0.381) (xy 0.3048 -0.37846) (xy 0.2286 -0.32766) (xy 0.19304 -0.25908)
+      (xy 0.18288 -0.14478) (xy 0.18034 -0.0889) (xy 0.18796 0.05334) (xy 0.21336 0.12446)
+      (xy 0.24638 0.13462) (xy 0.3683 0.15748) (xy 0.5334 0.21082) (xy 0.71374 0.28702)
+      (xy 0.8763 0.37338) (xy 0.9271 0.40386) (xy 1.04394 0.4826) (xy 1.13538 0.54102)
+      (xy 1.15824 0.55626) (xy 1.20396 0.5334) (xy 1.30048 0.4445) (xy 1.44526 0.2921)
+      (xy 1.62814 0.08636) (xy 1.84912 -0.17018) (xy 1.87706 -0.20828) (xy 2.54762 -1.0033)
+      (xy 2.4638 -1.14046) (xy 2.40284 -1.3081) (xy 2.38252 -1.51638) (xy 2.42062 -1.77292)
+      (xy 2.5273 -1.98628) (xy 2.68224 -2.1463) (xy 2.87782 -2.25044) (xy 3.09626 -2.29108)
+      (xy 3.32486 -2.26822) (xy 3.54838 -2.16916) (xy 3.71602 -2.02946) (xy 3.86334 -1.8161)
+      (xy 3.92684 -1.57988) (xy 3.92684 -1.57988)) (layer Dwgs.User) (width 0.00254))
+  )
   (gr_line (start 167.64 96.52) (end 167.64 68.58) (angle 90) (layer Edge.Cuts) (width 0.15))
